File: matrixdisplay/matrixdisplay.kicad_pcb (KiCad board)
At the start: 2 copper layers, 73 x 31 mm, 95 parts, among them J1 FILAS, J2 COLUMNAS, J3 SWD, J4 USART, J5 FILAS, J6 COL, SW1 BT1, SW2 BT2, SW2 P_ON, U1 STM32F051K8Ux

Commit message: Add better ARC logo
Parts:
- removed G*** (x2): LOGO, LOGO

Commit message: feat(matrixdisplay): update components to exclude from BOM and save components 3D bodies
Other:
- board text added: "ArcMaker ${VERSION}"
- board text removed: "ArcMaker v0.1"
Changed lines of the file:
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@@
 		)
 	)
+	(property "BRANCH" "master")
+	(property "BUILD_DATE" "2025-11-16")
+	(property "STATUS" "dirty")
+	(property "VERSION" "V0.0.2.3")
 	(net 0 "")
 	(net 1 "GND")
@@
 		)
 	)
-	(gr_text "ArcMaker v0.1"
-		(at 167.65 76.6 0)
+	(gr_text "ArcMaker\n${VERSION}"
+		(at 165 82.5 0)
 		(layer "B.SilkS")
 		(effects
 			(font
-				(size 1 1)
-				(thickness 0.2)
+				(size 0.75 1)
+				(thickness 0.1875)
 				(bold yes)
 			)
@@
 		)
 	)
-	(gr_text "ArcMaker v0.1"
+	(gr_text "ArcMaker\n${VERSION}"
 		(at 139.85 104.2 0)
 		(layer "B.SilkS")
